Commit message: Fix direction of one of the joints and add the gripper urdf

File: victor_description/urdf/iiwa14_med.xacro (robot description, xacro)
@@ -72,5 +72,5 @@
           <mesh filename="package://victor_description/meshes/iiwa14_med/visual/link_1.stl"/>
         </geometry>
-        <material name="Orange"/>
+        <material name="White"/>
       </visual>
       <collision>
@@ -79,5 +79,5 @@
           <mesh filename="package://victor_description/meshes/iiwa14_med/visual/link_1.stl"/>
         </geometry>
-        <material name="Orange"/>
+        <material name="White"/>
       </collision>
     </link>
@@ -107,5 +107,5 @@
           <mesh filename="package://victor_description/meshes/iiwa14_med/visual/A2_origin_updated.stl"/>
         </geometry>
-        <material name="Orange"/>
+        <material name="White"/>
       </visual>
       <collision>
@@ -114,5 +114,5 @@
           <mesh filename="package://victor_description/meshes/iiwa14_med/visual/link_2.stl"/>
         </geometry>
-        <material name="Orange"/>
+        <material name="White"/>
       </collision>
     </link>
@@ -142,5 +142,5 @@
           <mesh filename="package://victor_description/meshes/iiwa14_med/visual/A3_origin_updated.stl"/>
         </geometry>
-        <material name="Orange"/>
+        <material name="White"/>
       </visual>
       <collision>
@@ -149,5 +149,5 @@
           <mesh filename="package://victor_description/meshes/iiwa14_med/visual/link_3.stl"/>
         </geometry>
-        <material name="Orange"/>
+        <material name="White"/>
       </collision>
     </link>
@@ -177,5 +177,5 @@
           <mesh filename="package://victor_description/meshes/iiwa14_med/visual/A4_origin_updated.stl"/>
         </geometry>
-        <material name="Orange"/>
+        <material name="White"/>
       </visual>
       <collision>
@@ -184,5 +184,5 @@
           <mesh filename="package://victor_description/meshes/iiwa14_med/visual/link_4.stl"/>
         </geometry>
-        <material name="Orange"/>
+        <material name="White"/>
       </collision>
     </link>
@@ -208,16 +208,16 @@
       </inertial>
       <visual>
-        <origin xyz="0 0 0" rpy="0 0 0"/>
+        <origin xyz="0 0 0" rpy="0 0 3.1415"/>
         <geometry>
           <mesh filename="package://victor_description/meshes/iiwa14_med/visual/A5_origin_updated.stl"/>
         </geometry>
-        <material name="Orange"/>
-      </visual>
-      <collision>
-        <origin xyz="0 0 0" rpy="0 0 0"/>
+        <material name="White"/>
+      </visual>
+      <collision>
+        <origin xyz="0 0 0" rpy="0 0 3.1415"/>
         <geometry>
           <mesh filename="package://victor_description/meshes/iiwa14_med/visual/link_5.stl"/>
         </geometry>
-        <material name="Orange"/>
+        <material name="White"/>
       </collision>
     </link>
@@ -244,16 +244,16 @@
       </inertial>
       <visual>
-        <origin xyz="0 0 0.0607" rpy="3.1415 0 0"/>
+        <origin xyz="0 0 -0.0607" rpy="3.1415 3.1415 0"/>
         <geometry>
           <mesh filename="package://victor_description/meshes/iiwa14_med/visual/A6_origin_updated.stl"/>
         </geometry>
-        <material name="Orange"/>
-      </visual>
-      <collision>
-        <origin xyz="0 0 0.0607" rpy="3.1415 0 0"/>
+        <material name="White"/>
+      </visual>
+      <collision>
+        <origin xyz="0 0 -0.0607" rpy="3.1415 3.1415 0"/>
         <geometry>
           <mesh filename="package://victor_description/meshes/iiwa14_med/visual/link_6.stl"/>
         </geometry>
-        <material name="Orange"/>
+        <material name="White"/>
       </collision>
     </link>

File: victor_description/urdf/med.urdf.xacro (robot description, xacro)
@@ -13,3 +13,8 @@
     <origin xyz="0 0 0" rpy="0 0 0"/>
   </xacro:iiwa14_med>
+  <!-- wsg50 gripper -->
+  <xacro:include filename="$(find wsg_50_simulation)/urdf/wsg_50.urdf.xacro"/>
+  <xacro:wsg_50_xacro name="wsg50" parent="$(arg robot_name)_kuka_link_ee" finger_length="0.023" finger_tip="0">
+    <origin xyz="0 0 0" rpy="0 0 -1.5708"/>
+  </xacro:wsg_50_xacro>
 </robot>
