Commit message: Add med control and extend urdf to include gazebo control plugins as needed.

File: victor_description/urdf/med.urdf.xacro (robot description, xacro)
@@ -1,20 +1,29 @@
 <?xml version="1.0"?>
 <robot name="med" xmlns:xacro="http://www.ros.org/wiki/xacro">
-  <xacro:arg name="robot_name" default="med"/>
-  <xacro:arg name="kinematic_arms" default="0"/>
-  <xacro:arg name="hardware_interface" default="hardware_interface/PositionJointInterface"/>
-  <!-- Import Rviz colors -->
-  <xacro:include filename="$(find victor_description)/urdf/materials.xacro"/>
-  <!-- Make a base link. -->
-  <link name="$(arg robot_name)_base" type="fixed"/>
-  <!-- iiwa med arm -->
-  <xacro:include filename="$(find victor_description)/urdf/iiwa14_med.xacro"/>
-  <xacro:iiwa14_med hardware_interface="$(arg hardware_interface)" robot_name="$(arg robot_name)_kuka" parent="$(arg robot_name)_base" kinematic="$(arg kinematic_arms)">
-    <origin xyz="0 0 0" rpy="0 0 0"/>
-  </xacro:iiwa14_med>
-  <!-- wsg50 gripper -->
-  <xacro:include filename="$(find wsg_50_simulation)/urdf/wsg_50.urdf.xacro"/>
-  <xacro:wsg_50_xacro name="wsg50" parent="$(arg robot_name)_kuka_link_ee" finger_length="0.023" finger_tip="0">
-    <origin xyz="0 0 0" rpy="0 0 -1.5708"/>
-  </xacro:wsg_50_xacro>
+    <xacro:arg name="robot_name" default="med"/>
+    <xacro:arg name="kinematic_arms" default="0"/>
+    <xacro:arg name="hardware_interface" default="hardware_interface/PositionJointInterface"/>
+    <!-- Import Rviz colors -->
+    <xacro:include filename="$(find victor_description)/urdf/materials.xacro"/>
+    <!-- Make a base link. -->
+    <link name="$(arg robot_name)_base" type="fixed"/>
+    <!-- iiwa med arm -->
+    <xacro:include filename="$(find victor_description)/urdf/iiwa14_med.xacro"/>
+    <xacro:iiwa14_med hardware_interface="$(arg hardware_interface)" robot_name="$(arg robot_name)_kuka"
+                      parent="$(arg robot_name)_base" kinematic="$(arg kinematic_arms)">
+        <origin xyz="0 0 0" rpy="0 0 0"/>
+    </xacro:iiwa14_med>
+    <!-- wsg50 gripper -->
+    <xacro:include filename="$(find wsg_50_simulation)/urdf/wsg_50.urdf.xacro"/>
+    <xacro:wsg_50_xacro name="wsg50" parent="$(arg robot_name)_kuka_link_ee" finger_length="0.023"
+                        finger_tip="0" hardware_interface="$(arg hardware_interface)">
+        <origin xyz="0 0 0" rpy="0 0 -1.5708"/>
+    </xacro:wsg_50_xacro>
+    <!-- Gazebo setup -->
+    <xacro:include filename="$(find victor_description)/urdf/gazebo_utilities.xacro"/>
+    <!-- Load Gazebo lib and set the robot namespace -->
+    <xacro:add_gazebo_control_plugin robot_namespace="$(arg robot_name)"/>
+    <xacro:add_moveit_planning_scene_plugin robot_namespace="$(arg robot_name)" root_frame_id="$(arg robot_name)_base"/>
+    <!-- Rigidly attach Med to the Gazebo world -->
+    <xacro:add_gazebo_fixed_link base_link="$(arg robot_name)_base"/>
 </robot>

File: victor_description/urdf/victor.urdf.xacro (robot description, xacro)
@@ -39,21 +39,21 @@
     </link>
     <!-- arm to gripper adapter -->
-    <!-- <xacro:include filename="$(find victor_description)/urdf/iiwa7_to_robotiq_adapter.xacro"/> -->
-    <!-- <xacro:iia7_to_robotiq_adapter parent="$(arg robot_name)_left_arm_flange" prefix="$(arg robot_name)_left"> -->
-    <!--     <origin xyz="0 0 -0.01" rpy="0 0 0"/> -->
-    <!-- </xacro:iia7_to_robotiq_adapter> -->
-    <!-- <xacro:iia7_to_robotiq_adapter parent="$(arg robot_name)_right_arm_flange" prefix="$(arg robot_name)_right"> -->
-    <!--     <origin xyz="0 0 -0.01" rpy="0 0 0"/> -->
-    <!-- </xacro:iia7_to_robotiq_adapter> -->
-    <!-- <!-\- Robotiq grippers -\-> -->
-    <!-- <xacro:if value="${gripper == 'kinematic_robotiq'}"> -->
-    <!--     <xacro:include filename="$(find victor_description)/urdf/kinematic_robotiq_grippers.xacro"/> -->
-    <!-- </xacro:if> -->
-    <!-- <xacro:if value="${gripper == 'robotiq'}"> -->
-    <!--     <xacro:include filename="$(find victor_description)/urdf/robotiq_grippers.xacro"/> -->
-    <!-- </xacro:if> -->
-    <!-- <!-\- Define additional links as "tools", which are useful for planning and getting transforms -\-> -->
-    <!-- <xacro:include filename="$(find victor_description)/urdf/robotiq_pinch_grasp_tools.xacro"/> -->
-    <!-- <xacro:robotiq_pinch_grasp_tools robot_name="$(arg robot_name)"/> -->
+     <xacro:include filename="$(find victor_description)/urdf/iiwa7_to_robotiq_adapter.xacro"/>
+     <xacro:iia7_to_robotiq_adapter parent="$(arg robot_name)_left_arm_flange" prefix="$(arg robot_name)_left">
+         <origin xyz="0 0 -0.01" rpy="0 0 0"/>
+     </xacro:iia7_to_robotiq_adapter>
+     <xacro:iia7_to_robotiq_adapter parent="$(arg robot_name)_right_arm_flange" prefix="$(arg robot_name)_right">
+         <origin xyz="0 0 -0.01" rpy="0 0 0"/>
+     </xacro:iia7_to_robotiq_adapter>
+     <!-- Robotiq grippers -->
+     <xacro:if value="${gripper == 'kinematic_robotiq'}">
+         <xacro:include filename="$(find victor_description)/urdf/kinematic_robotiq_grippers.xacro"/>
+     </xacro:if>
+     <xacro:if value="${gripper == 'robotiq'}">
+         <xacro:include filename="$(find victor_description)/urdf/robotiq_grippers.xacro"/>
+     </xacro:if>
+     <!-- Define additional links as "tools", which are useful for planning and getting transforms -->
+     <xacro:include filename="$(find victor_description)/urdf/robotiq_pinch_grasp_tools.xacro"/>
+     <xacro:robotiq_pinch_grasp_tools robot_name="$(arg robot_name)"/>
     <!-- Add Gazebo properties for whole robot -->
     <xacro:include filename="$(find victor_description)/urdf/victor.gazebo.xacro"/>
